File: edge-connector.kicad_sch (KiCad schematic)
At the start: 1 part, among them J2 PCB-Edge_DC-SCM-2.1_2x84_Rev-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

Commit message: [#100720] Route high speeds
Parts:
- J2: footprint antmicro-footprints:PCB-Edge_DC-SCM_2x84_Rev-1-0 -> antmicro-footprints:PCB-Edge_DC-SCM-2.1_2x84_Rev-1-1
Connections:
- net DC_SCM_I2C_I3C16.SCL: now also J2.A52 (I2C_I3C_1V8_16_SDA); no longer J2.A51 (I2C_I3C_1V8_16_SCL)
- net DC_SCM_I2C_I3C16.SDA: now also J2.A51 (I2C_I3C_1V8_16_SCL); no longer J2.A52 (I2C_I3C_1V8_16_SDA)

Commit message: [#100720] Start USB section
Parts:
- added R132, R133, R141, R142, R143, R144: R_0R_0402, antmicro-footprints:R_0402_1005Metric, symbol antmicroResistors0402:R_0R_0402
Connections:
- net DC-SCM_CLK_100M_1.CLK+: now also R143.1
- net DC-SCM_CLK_100M_1.CLK-: now also R144.1
- net PCIE_LOCAL_USB_TX0-: now reaches J2.A65 (PCIE_HPMROOT_SCM_HPM_5_DN)
- net PCIE_LOCAL_USB_TX0-: now also R142.1
- net PCIE_LOCAL_USB_TX0+: now reaches J2.A66 (PCIE_HPMROOT_SCM_HPM_5_DP)
- net PCIE_LOCAL_USB_TX0+: now also R141.1
- net PCIE_LOCAL_USB_RX0-: now reaches J2.B65 (PCIE_HPMROOT_HPM_SCM_5_DN)
- net PCIE_LOCAL_USB_RX0-: now also R133.1
- net PCIE_LOCAL_USB_RX0+: now reaches J2.B66 (PCIE_HPMROOT_HPM_SCM_5_DP)
- net PCIE_LOCAL_USB_RX0+: now also R132.1
- new net DC-SCM_CLK_100M_USB.CLK+: R143.2
- new net DC-SCM_CLK_100M_USB.CLK-: R144.2
- new net DC-SCM_PCIE_LOCAL_USB.RX0+: R132.2
- new net DC-SCM_PCIE_LOCAL_USB.RX0-: R133.2
- new net DC-SCM_PCIE_LOCAL_USB.TX0+: R141.2
- new net DC-SCM_PCIE_LOCAL_USB.TX0-: R142.2
- no-connect marks 4 -> 0
Other:
- moved on the sheet: J2D

Commit message: [#100720] Apply post review changes
Parts:
- removed R132, R133, R141, R142, R143, R144: R_0R_0402, antmicro-footprints:R_0402_1005Metric, symbol antmicroResistors0402:R_0R_0402
Connections:
- net PCIE_LOCAL_USB_RX0+ is gone; now on net DC-SCM_PCIE_LOCAL_USB.TX0+: J2.B66 (PCIE_HPMROOT_HPM_SCM_5_DP)
- net PCIE_LOCAL_USB_RX0- is gone; now on net DC-SCM_PCIE_LOCAL_USB.TX0-: J2.B65 (PCIE_HPMROOT_HPM_SCM_5_DN)
- net PCIE_LOCAL_USB_TX0+ is gone; now on net DC-SCM_PCIE_LOCAL_USB.RX0+: J2.A66 (PCIE_HPMROOT_SCM_HPM_5_DP)
- net PCIE_LOCAL_USB_TX0- is gone; now on net DC-SCM_PCIE_LOCAL_USB.RX0-: J2.A65 (PCIE_HPMROOT_SCM_HPM_5_DN)
- net DC_SCM_I2C_I3C16.SCL: now also J2.A51 (I2C_I3C_1V8_16_SCL); no longer J2.A52 (I2C_I3C_1V8_16_SDA)
- net DC_SCM_I2C_I3C16.SDA: now also J2.A52 (I2C_I3C_1V8_16_SDA); no longer J2.A51 (I2C_I3C_1V8_16_SCL)
