File: dc-scm-server-integration-dc-scm-debug-interposer.kicad_pcb (KiCad board)
At the start: 6 copper layers, 90 x 62.3 mm, 166 parts, among them J1 Socket_DC-SCM-2.1_2x84_Rev-1-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, J10 PinHeader_2x5_P2.54mm_SMD, J11 PinHeader_2x5_P2.54mm_SMD, J12 PinHeader_2x5_P2.54mm_SMD, J13 PinHeader_2x5_P2.54mm_SMD, J15 Socket_SOP2-16_ACA-SPI-006-K0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, J16 Socket_SOP2-16_ACA-SPI-006-K0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, J17 PinHeader_2x5_P2.54mm_SMD, J2 PCB-Edge_DC-SCM-2.1_2x84_Rev-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, J3 PinHeader_2x5_P2.54mm_SMD, J4 PinHeader_2x5_P2.54mm_SMD, J5 PinHeader_2x5_P2.54mm_SMD, J6 PinHeader_2x5_P2.54mm_SMD, J7 PinHeader_2x5_P2.54mm_SMD, J9 PinHeader_2x5_P2.54mm_SMD, Q3 DMG1012T-7, U1 TLV76701_WSON

Commit message: [#100720] Continue routing low speeds
Parts:
- moved R13 0.53 mm to (145.7, 80.2)
- moved R99 0.12 mm to (148.6, 80.2), turned to -90 degrees
- turned R19 to 90 degrees
Routing:
- net /DC-SCI edge connector/DC_SCM_QSPI.IO2: track 0.00 -> 98.5 mm, vias 0 -> 5
- net /DC-SCI edge connector/DC_SCM_QSPI.IO1: track 0.00 -> 95.0 mm, vias 0 -> 5
- net /DC-SCI edge connector/DC_SCM_QSPI.IO0: track 0.00 -> 93.0 mm, vias 0 -> 5
- net /DC-SCI edge connector/DC_SCM_QSPI.~{CS1}: track 0.00 -> 92.1 mm, vias 0 -> 4
- net /DC-SCI edge connector/DC_SCM_QSPI.IO3: track 0.00 -> 84.4 mm, vias 0 -> 5
- net /DC-SCI edge connector/DC_SCM_QSPI.SCK: track 0.00 -> 79.0 mm, vias 0 -> 2
- net /DC-SCI edge connector/DC_SCM_QSPI.~{CS0}: track 0.00 -> 75.8 mm, vias 0 -> 4
- net /DC-SCI edge connector/DC_SCM_I2C2.SDA: track 0.00 -> 67.0 mm, vias 0 -> 2
- net /DC-SCI edge connector/DC_SCM_I2C2.SCL: track 0.00 -> 64.9 mm, vias 0 -> 2
- net /DC-SCI edge connector/DC_SCM_PRSNT1_N: track 0.00 -> 59.5 mm, vias 0 -> 1
- net /DC-SCI edge connector/DC_SCM_JTAG.TCK: track 0.00 -> 56.4 mm, vias 0 -> 1
- net /DC-SCI edge connector/DC_SCM_JTAG.TDO: track 0.00 -> 54.6 mm, vias 0 -> 1
- net /DC-SCI edge connector/DC_SCM_P3V0: track 0.00 -> 53.0 mm, vias 0 -> 3
- net /DC-SCI edge connector/~{PCIE_HPM_SCM_PERST}: track 0.00 -> 51.8 mm
- net /DC-SCI edge connector/DC_SCM_STBY_RDY: track 0.00 -> 10.4 mm, vias 0 -> 2
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
Commit message: [#100720] Route power
Parts:
- R1: value R_0R_0402 -> R_0R_22.4A_0603; footprint antmicro-footprints:R_0402_1005Metric -> antmicro-footprints:R_0603_1608Metric
- moved R55 0.80 mm to (125.8, 78.2)
- moved C1 0.76 mm to (101.7, 107.1)
- moved C2 0.76 mm to (106.8, 107.1)
- moved R128 0.76 mm to (110.8, 107.1)
- moved R131 0.76 mm to (107.8, 107.1)
- moved R132 0.76 mm to (108.8, 107.1), turned to -90 degrees
- moved R133 0.76 mm to (109.8, 107.1), turned to 90 degrees
- moved U1 0.76 mm to (104.2, 107.0)
- moved R54 0.45 mm to (127.1, 78.2)
- moved R1 0.11 mm to (130.3, 78.2)
Connections:
- net Net-(J1A-P12V_AUX-PadA1) renamed /DC-SCI gold fingers connector/12V_AUX
Routing:
- net +1V8: track 0.00 -> 106.3 mm, vias 0 -> 6
- net /DC-SCI edge connector/DC_SCM_ESPI.~{ALERT0}: track 0.00 -> 71.5 mm, vias 0 -> 3
- net /DC-SCI edge connector/DC_SCM_ESPI.IO0: track 0.00 -> 70.5 mm, vias 0 -> 3
- net /DC-SCI edge connector/DC_SCM_ESPI.IO3: track 0.00 -> 68.1 mm, vias 0 -> 3
- net /DC-SCI edge connector/DC_SCM_ESPI.IO2: track 0.00 -> 67.5 mm, vias 0 -> 3
- net /DC-SCI edge connector/DC_SCM_ESPI.~{RESET}: track 0.00 -> 65.5 mm, vias 0 -> 3
- net /DC-SCI edge connector/DC_SCM_ESPI.~{CS0}: track 0.00 -> 64.2 mm, vias 0 -> 3
- net /DC-SCI edge connector/DC_SCM_ESPI.IO1: track 0.00 -> 60.8 mm, vias 0 -> 2
- net /DC-SCI edge connector/DC_SCM_ESPI.SCK: track 0.00 -> 60.0 mm, vias 0 -> 2
- net /DC-SCI edge connector/DC_SCM_I2C_I3C17.SDA: track 3.85 -> 62.9 mm, vias 0 -> 4
- net /DC-SCI edge connector/DC_SCM_PECI: track 0.00 -> 55.9 mm, vias 0 -> 1
- net /DC-SCI edge connector/DC_SCM_I2C_I3C17.SCL: track 1.51 -> 56.8 mm, vias 0 -> 3
- net /DC-SCI edge connector/PECI_VREF_HPM_SCM: track 0.00 -> 47.5 mm, vias 0 -> 3
- net /DC-SCI edge connector/DC_SCM_P3V0: track 53.0 -> 99.9 mm, vias 3 -> 4
- net /DC-SCI edge connector/DC_SCM_STBY_RDY: track 10.4 -> 50.5 mm, vias 2 -> 3
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- added copper zone on B.Cu, net /DC-SCI edge connector/DC_SCM_12V_AUX
- added copper zone on In3.Cu, net /DC-SCI edge connector/DC_SCM_12V_AUX
- added copper zone on B.Cu, net /DC-SCI gold fingers connector/12V_AUX

Commit message: [#100720] Continue routing low speeds
Parts:
- R67, R68, R69, R70: moved to B.Cu
- moved R99 23.6 mm to (125.0, 80.6)
- moved R2 23.1 mm to (123.8, 80.6)
- moved R18 23.1 mm to (124.4, 82.6)
- moved R3 23.1 mm to (122.6, 80.6)
- moved R19 22.7 mm to (125.7, 82.6)
- moved R13 22.6 mm to (123.2, 82.6)
- moved R55 5.84 mm to (122.0, 82.6)
- moved R75 4.35 mm to (156.0, 80.2)
- moved R76 4.35 mm to (156.6, 78.2)
- moved R77 4.30 mm to (157.2, 80.2)
- moved R78 4.30 mm to (157.8, 78.2)
- moved R68 2.05 mm to (160.4, 80.2)
- moved R67 2.05 mm to (159.9, 82.2)
- moved R69 2.05 mm to (161.1, 82.2)
- moved R70 2.05 mm to (161.7, 80.2)
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Routing:
- net /DC-SCI edge connector/~{DC_SCM_INTRUSION}: track 9.90 -> 68.2 mm, vias 2 -> 3
- net /DC-SCI edge connector/DC_SCM_P3V0: track 99.9 -> 43.3 mm, vias 4 -> 2
- net /DC-SCI edge connector/DC_SCM_PRSNT0_N: track 52.6 -> 86.4 mm, vias 0 -> 2
- net Net-(J1A-HPM_SCM_INTRUSION_N): track 0.00 -> 30.3 mm, vias 0 -> 2
- net Net-(J1A-HPM_SCM_STBY_RDY): track 0.00 -> 28.4 mm, vias 0 -> 2
- net Net-(J1A-P3V0_HPM_SCM_BAT): track 0.00 -> 28.4 mm, vias 0 -> 2
- net Net-(J1B-I2C_3V3_2_SDA): track 6.46 -> 27.9 mm, vias 0 -> 2
- net Net-(J1B-I2C_3V3_2_SCL): track 8.48 -> 27.8 mm, vias 0 -> 2
- net Net-(J1D-PCIE_HPM_SCM_PERST_N): track 8.49 -> 26.2 mm, vias 0 -> 2
- net /DC-SCI edge connector/DC_SCM_STBY_RDY: track 50.5 -> 67.5 mm, vias 3 -> 2
- net Net-(J1B-I2C_I3C_1V8_15_SCL): track 0.00 -> 14.6 mm, vias 0 -> 2
- net Net-(J1B-I2C_I3C_1V8_14_SCL): track 0.00 -> 13.6 mm, vias 0 -> 2
- net Net-(J1B-I2C_I3C_1V8_15_SDA): track 0.00 -> 12.9 mm, vias 0 -> 2
- net /DC-SCI edge connector/DC_SCM_I2C2.SCL: track 64.9 -> 77.7 mm, vias 2 -> 3
- net Net-(J1B-I2C_I3C_1V8_14_SDA): track 0.00 -> 12.5 mm, vias 0 -> 2
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Other:
- board size 90 x 62.3 mm -> 90 x 62.4 mm
