File: peripherals.kicad_sch (KiCad schematic)
At the start: 48 parts, among them J12 PinHeader_2x5_P1.27mm_SMD, J13 PinHeader_2x5_P1.27mm_SMD, J14 PinHeader_2x5_P1.27mm_SMD, J15 PinHeader_2x5_P1.27mm_SMD, J16 PinHeader_2x5_P1.27mm_SMD, J20 PinHeader_2x5_P1.27mm_SMD, J3 Socket_SOP2-16_ACA-SPI-006-K0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, J4 Socket_SOP2-16_ACA-SPI-006-K0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, J6 PinHeader_2x10_P1.27mm_SMD_Sh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, J8 PinHeader_1x2_P1.27mm_Drill0.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, J9 PinHeader_2x5_P1.27mm_SMD_Shr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, Q2 DMG1012T-7, Q3 DMG1012T-7

Commit message: [#100720] Add DCDC
Parts:
- removed J3, J4: Socket_SOP2-16_ACA-SPI-006-K01_CUSTOM, antmicro-footprints:Socket_SOP2-16_ACA-SPI-006-K01, symbol antmicroMechanicalParts:Socket_SOP2-16_ACA-SPI-006-K01_CUSTOM
- removed R12, R17: R_220R_0402, antmicro-footprints:R_0402_1005Metric, symbol antmicroResistors0402:R_220R_0402
- removed R131: R_10k_0402, antmicro-footprints:R_0402_1005Metric, symbol antmicroResistors0402:R_10k_0402
- added J21, J22, J23: PinHeader_2x5_P1.27mm_SMD, antmicro-footprints:PinHeader_2x5_P1.27mm_SMD, symbol antmicroGenericPinHeaders:PinHeader_2x5_P1.27mm_SMD
- added R140, R141: R_10k_0402, antmicro-footprints:R_0402_1005Metric, symbol antmicroResistors0402:R_10k_0402
- added TP30, TP31, TP32, TP33, TP34, TP35: TP_1mm_SMD, antmicro-footprints:TP_SMD_1mm, symbol antmicroTestPoints:TP_1mm_SMD
Connections:
- net +3V3: now also R140.2, R141.2
- net DC_SCM_12V_AUX: now also J21.1
- net DC_SCM_HPM_FRU: now also J21.6
- net DC_SCM_NC-SI.CRS_DV: now also J23.3
- net DC_SCM_NC-SI.REF_CLK: now also J23.1
- net DC_SCM_NC-SI.RXD0: now also J23.5
- net DC_SCM_NC-SI.RXD1: now also J23.7
- net DC_SCM_NC-SI.TXD0: now also J23.4
- net DC_SCM_NC-SI.TXD1: now also J23.6
- net DC_SCM_NC-SI.TX_EN: now also J23.2
- net DC_SCM_P3V0: now also J21.3
- net DC_SCM_PRSNT0_N: now also J21.5
- net DC_SCM_PRSNT1_N: now also J21.7
- net DC_SCM_QSPI.IO0: now also J22.1
- net DC_SCM_QSPI.IO1: now also J22.3
- net DC_SCM_QSPI.IO2: now also J22.5
- net DC_SCM_QSPI.IO3: now also J22.7
- net DC_SCM_QSPI.SCK: now also J22.6
- net DC_SCM_QSPI.~{CS0}: now also J22.2
- net DC_SCM_QSPI.~{CS1}: now also J22.4
- net DC_SCM_UART.RX: now also J21.2
- net DC_SCM_UART.TX: now also J21.4
- net DC_SCM_USB1.D+: now also TP30.1
- net DC_SCM_USB1.D-: now also TP31.1
- net DC_SCM_USB2.D+: now also TP32.1
- net DC_SCM_USB2.D-: now also TP33.1
- net GND: now also J22.10, J22.8, J22.9, J23.10, J23.8, J23.9
- net PECI_VREF_HPM_SCM: now also J21.8
- net ~{DC_SCM_INTRUSION}: now also J21.9
- net ~{DC_SCM_SPI_SCMCNTRL_IRQ0}: now also J21.10
- net at D4.2 (A): now also R140.1
- net at D10.2 (A): now also R141.1
- net at J6.15: now also TP34.1
- net at J6.16: now also TP35.1
Other:
- note added: "Misc + UART"
- note added: "NC-SI"
- note added: "PCIe"
- note added: "QSPI"
- note added: "USB"
- moved on the sheet: D10, D4, J12, J13, J14, J15, J16, J20, J6, J8, J9, Q2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

Commit message: [#100720] Swap DCDC for LDO
Parts:
- removed J8: PinHeader_1x2_P1.27mm_Drill0.7mm, antmicro-footprints:PinHeader_1x2_P1.27mm_Drill0.7mm, symbol antmicroGenericPinHeaders:PinHeader_1x2_P1.27mm_Drill0.7mm
- added TP36: TP_1mm_SMD, antmicro-footprints:TP_SMD_1mm, symbol antmicroTestPoints:TP_1mm_SMD
- renumbered D4 to D1, D10 to D2
Connections:
- net +3V3 is gone; now on net DC_SCM_12V_AUX: R140.2, R141.2
- net GND: no longer J22.10, J22.8, J23.10, J23.8
- net 3V3_TEST: now reaches J9.1
- net 3V3_TEST: now also TP36.1
- new net +1V8: J22.10, J22.8, J23.10, J23.8

Commit message: [#100720] Finish schematic, clean ERC
Parts:
- added J17: PinHeader_2x5_P1.27mm_SMD, antmicro-footprints:PinHeader_2x5_P1.27mm_SMD, symbol antmicroGenericPinHeaders:PinHeader_2x5_P1.27mm_SMD
Connections:
- net GND: now also J17.10, J17.5, J17.6, J17.9
- new net DC_SCM_I2C0.SCL: J17.1
- new net DC_SCM_I2C0.SDA: J17.2
- new net DC_SCM_I2C5.SCL: J17.3
- new net DC_SCM_I2C5.SDA: J17.4
- new net DC_SCM_I2C6.SCL: J17.7
- new net DC_SCM_I2C6.SDA: J17.8
Other:
- moved on the sheet: D1, D2, J12, J13, J14, J15, J6, Q2, Q3, R140, R141, R56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

Commit message: [#100720] Reannotate
Parts:
- renumbered J20 to J10, J22 to J11, J23 to J12, J21 to J13, J9 to J14, J17 to J3, J12 to J4, J13 to J5, J14 to J6, J15 to J7, J6 to J8, J16 to J9, Q2 to Q1, Q3 to Q2, R140 to R128, R56 to R129, R141 to R130, TP34 to TP1, TP8 to TP10, TP9 to TP11, TP10 to TP12, TP11 to TP13, TP12 to TP14, TP13 to TP15, TP14 to TP16, TP15 to TP17, TP16 to TP18, TP17 to TP19, TP35 to TP2, TP18 to TP20, TP19 to TP21, TP20 to TP22, TP21 to TP23, TP22 to TP24, TP23 to TP25, TP24 to TP26, TP25 to TP27, TP26 to TP28, TP27 to TP29, TP1 to TP3, TP28 to TP30, TP29 to TP31, TP30 to TP32, TP31 to TP33, TP32 to TP34, TP33 to TP35, TP2 to TP4, TP3 to TP5, TP4 to TP6, TP5 to TP7, TP6 to TP8, TP7 to TP9

Commit message: [#100720] Place connectors
Parts:
- removed D1, D2: LED_G_0402_VLMTG1500-GS08, antmicro-footprints:LED_0402_1005Metric_G, symbol antmicroLEDIndicationDiscrete:LED_G_0402_VLMTG1500-GS08
- removed J10, J11, J12, J13, J3, J4, J5, J6, J7, J9: PinHeader_2x5_P1.27mm_SMD, antmicro-footprints:PinHeader_2x5_P1.27mm_SMD, symbol antmicroGenericPinHeaders:PinHeader_2x5_P1.27mm_SMD
- removed J14: PinHeader_2x5_P1.27mm_SMD_Shrouded, antmicro-footprints:PinHeader_2x5_P1.27mm_SMD_Shrouded, symbol antmicroGenericPinHeaders:PinHeader_2x5_P1.27mm_SMD_Shrouded
- removed J8: PinHeader_2x10_P1.27mm_SMD_Shrouded, antmicro-footprints:PinHeader_2x10_P1.27mm_SMD_Shrouded, symbol antmicroGenericPinHeaders:PinHeader_2x10_P1.27mm_SMD_Shrouded
- removed Q1, Q2: DMG1012T-7, antmicro-footprints:SOT-523, symbol antmicroTransistorsFETsMOSFETsSingle:DMG1012T-7
- removed R128, R130: R_10k_0402, antmicro-footprints:R_0402_1005Metric, symbol antmicroResistors0402:R_10k_0402
- removed R129: R_100k_0402, antmicro-footprints:R_0402_1005Metric, symbol antmicroResistors0402:R_100k_0402
- removed TP1, TP10, TP11, TP12, TP13, TP14, TP15, TP16, TP17, TP18, TP19, TP2, TP20, TP21, TP22, TP23, TP24, TP25, TP26, TP27, TP28, TP29, TP3, TP30, TP31, TP32, TP33, TP34, TP35, TP36, TP4, TP5, TP6, TP7, TP8, TP9: TP_1mm_SMD, antmicro-footprints:TP_SMD_1mm, symbol antmicroTestPoints:TP_1mm_SMD
- added J10, J11, J12, J13, J17, J3, J4, J5, J6, J7, J9: PinHeader_2x5_P2.54mm_SMD, antmicro-footprints:PinHeader_2x5_P2.54mm_SMD, symbol antmicroGenericPinHeaders:PinHeader_2x5_P2.54mm_SMD
Connections:
- net +1V8: now also J11.10, J11.8, J12.10, J17.2
- net DC_SCM_12V_AUX: now also J17.1
- net DC_SCM_ESPI.IO0: now also J10.9
- net DC_SCM_ESPI.IO1: now also J10.2
- net DC_SCM_ESPI.IO2: now also J10.4
- net DC_SCM_ESPI.IO3: now also J10.8
- net DC_SCM_ESPI.SCK: now also J10.1
- net DC_SCM_ESPI.~{ALERT0}: now also J10.10
- net DC_SCM_ESPI.~{CS0}: now also J10.3
- net DC_SCM_ESPI.~{RESET}: now also J10.7
- net DC_SCM_HPM_FRU: now also J17.8
- net DC_SCM_I2C0.SCL: now also J3.1
- net DC_SCM_I2C0.SDA: now also J3.2
- net DC_SCM_I2C1.SCL: now also J4.1
- net DC_SCM_I2C1.SDA: now also J4.2
- net DC_SCM_I2C2.SCL: now also J4.3
- net DC_SCM_I2C2.SDA: now also J4.4
- net DC_SCM_I2C3.SCL: now also J4.7
- net DC_SCM_I2C3.SDA: now also J4.8
- net DC_SCM_I2C4.SCL: now also J4.9
- net DC_SCM_I2C4.SDA: now also J4.10
- net DC_SCM_I2C5.SCL: now also J3.3
- net DC_SCM_I2C5.SDA: now also J3.4
- net DC_SCM_I2C6.SCL: now also J3.7
- net DC_SCM_I2C6.SDA: now also J3.8
- net DC_SCM_I2C7.SCL: now also J5.1
- net DC_SCM_I2C7.SDA: now also J5.2
- net DC_SCM_I2C8.SCL: now also J5.3
- net DC_SCM_I2C8.SDA: now also J5.4
- net DC_SCM_I2C9.SCL: now also J5.7
- net DC_SCM_I2C9.SDA: now also J5.8
- net DC_SCM_I2C_I3C12.SCL: now also J5.9
- net DC_SCM_I2C_I3C12.SDA: now also J5.10
- net DC_SCM_I2C_I3C13.SCL: now also J6.1
- net DC_SCM_I2C_I3C13.SDA: now also J6.2
- net DC_SCM_I2C_I3C14.SCL: now also J6.3
- net DC_SCM_I2C_I3C14.SDA: now also J6.4
- net DC_SCM_I2C_I3C15.SCL: now also J6.7
- net DC_SCM_I2C_I3C15.SDA: now also J6.8
- net DC_SCM_I2C_I3C16.SCL: now also J6.9
- net DC_SCM_I2C_I3C16.SDA: now also J6.10
- net DC_SCM_I2C_I3C17.SCL: now also J7.1
- net DC_SCM_I2C_I3C17.SDA: now also J7.2
- net DC_SCM_I2C_I3C18.SCL: now also J7.6
- net DC_SCM_I2C_I3C18.SDA: now also J7.4
- net DC_SCM_I2C_I3C19.SCL: now also J7.10
- net DC_SCM_I2C_I3C19.SDA: now also J7.8
- net DC_SCM_JTAG.TCK: now also J13.3
- net DC_SCM_JTAG.TDI: now also J13.7
- net DC_SCM_JTAG.TDO: now also J13.5
- net DC_SCM_JTAG.TMS: now also J13.1
- net DC_SCM_JTAG.TRST: now also J13.9
- net DC_SCM_NC-SI.CRS_DV: now also J12.3
- net DC_SCM_NC-SI.REF_CLK: now also J12.1
- net DC_SCM_NC-SI.RXD0: now also J12.5
- net DC_SCM_NC-SI.RXD1: now also J12.7
- net DC_SCM_NC-SI.TXD0: now also J12.4
- net DC_SCM_NC-SI.TXD1: now also J12.6
- net DC_SCM_NC-SI.TX_EN: now also J12.2
- net DC_SCM_P3V0: now also J17.3
- net DC_SCM_PECI: now also J17.4
- net DC_SCM_PRSNT0_N: now also J13.6
- net DC_SCM_PRSNT1_N: now also J13.8
- net DC_SCM_QSPI.IO0: now also J11.1
- net DC_SCM_QSPI.IO1: now also J11.3
- net DC_SCM_QSPI.IO2: now also J11.5
- net DC_SCM_QSPI.IO3: now also J11.7
- net DC_SCM_QSPI.SCK: now also J11.6
- net DC_SCM_QSPI.~{CS0}: now also J11.2
- net DC_SCM_QSPI.~{CS1}: now also J11.4
- net DC_SCM_SPI_SCMCNTRL.DI: now also J9.10
- net DC_SCM_SPI_SCMCNTRL.DO: now also J9.8
- net DC_SCM_SPI_SCMCNTRL.SCK: now also J9.2
- net DC_SCM_SPI_SCMCNTRL.~{CS0}: now also J9.4
- net DC_SCM_SPI_SCMCNTRL.~{CS1}: now also J9.6
- net DC_SCM_STBY_EN: now also J17.6
- net DC_SCM_STBY_RDY: now also J17.5
- net DC_SCM_TPM_SPI.DI: now also J9.5
- net DC_SCM_TPM_SPI.DO: now also J9.7
- net DC_SCM_TPM_SPI.SCK: now also J9.1
- net DC_SCM_TPM_SPI.~{CS0}: now also J9.3
- net DC_SCM_UART.RX: now also J13.2
- net DC_SCM_UART.TX: now also J13.4
- net GND: now also J10.5, J10.6, J11.9, J12.8, J12.9, J3.10, J3.5, J3.6, J3.9, J4.5, J4.6, J5.5, J5.6, J6.5, J6.6, J7.3, J7.5, J7.7, J7.9, J9.9
- net PECI_VREF_HPM_SCM: now also J17.10
- net ~{DC_SCM_INTRUSION}: now also J13.10
- net ~{DC_SCM_SPI_SCMCNTRL_IRQ0}: now also J17.9
- net ~{DC_SCM_STBY_RST}: now also J17.7
- no-connect marks 2 -> 0
Other:
- note added: "Misc + UART + JTAG"
- note added: "Miscellaneous"
- note removed: "Diff pairs aligned to keep pair cables next to each other in IDC cable"
- note removed: "JTAG"
- note removed: "LTPI"
- note removed: "LTPI LEDs"
- note removed: "Misc + UART"
- note removed: "PCIe"
- note removed: "USB"

Commit message: [#100720] Finish silkscreen
Connections:
- net DC_SCM_12V_AUX: now also J17.5; no longer J17.1
- net DC_SCM_ESPI.IO0: now also J10.7; no longer J10.9
- net DC_SCM_ESPI.IO3: now also J10.6; no longer J10.8
- net DC_SCM_ESPI.~{ALERT0}: now also J10.8; no longer J10.10
- net DC_SCM_ESPI.~{RESET}: now also J10.5; no longer J10.7
- net DC_SCM_STBY_RDY: now also J17.7; no longer J17.5
- net GND: now also J10.10, J10.9, J17.1; no longer J10.5, J10.6, J9.9
- net ~{DC_SCM_SPI_SCMCNTRL_IRQ0}: now also J9.9; no longer J17.9
- net ~{DC_SCM_STBY_RST}: now also J17.9; no longer J17.7
Changed lines of the file:
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@@
 	)
 	(bus_entry
-		(at 212.09 96.52)
+		(at 212.09 93.98)
 		(size 1.27 1.27)
 		(stroke
@@
 	)
 	(bus_entry
-		(at 292.1 93.98)
+		(at 292.1 91.44)
 		(size -1.27 1.27)
 		(stroke
@@
 	)
 	(bus_entry
-		(at 292.1 96.52)
+		(at 292.1 93.98)
 		(size -1.27 1.27)
 		(stroke
@@
 	)
 	(bus_entry
-		(at 212.09 93.98)
+		(at 212.09 91.44)
 		(size 1.27 1.27)
 		(stroke
@@
 	(wire
 		(pts
-			(xy 100.33 195.58) (xy 102.87 195.58)
+			(xy 100.33 198.12) (xy 102.87 198.12)
 		)
 		(stroke
@@
 	(wire
 		(pts
-			(xy 100.33 187.96) (xy 102.87 187.96)
+			(xy 100.33 193.04) (xy 102.87 193.04)
 		)
 		(stroke
@@
 	(wire
 		(pts
-			(xy 256.54 97.79) (xy 290.83 97.79)
+			(xy 256.54 95.25) (xy 290.83 95.25)
 		)
 		(stroke
@@
 	(wire
 		(pts
+			(xy 245.11 97.79) (xy 246.38 97.79)
+		)
+		(stroke
+			(width 0)
+			(type default)
+		)
+	)
+	(wire
+		(pts
 			(xy 215.9 138.43) (xy 246.38 138.43)
 		)
@@
 		)
 	)
-	(bus
-		(pts
-			(xy 292.1 88.9) (xy 292.1 93.98)
-		)
-		(stroke
-			(width 0)
-			(type default)
-		)
-	)
 	(wire
 		(pts
@@
 	(bus
 		(pts
-			(xy 212.09 93.98) (xy 212.09 96.52)
+			(xy 212.09 88.9) (xy 212.09 93.98)
 		)
 		(stroke
@@
 	(bus
 		(pts
-			(xy 212.09 88.9) (xy 212.09 93.98)
-		)
-		(stroke
-			(width 0)
-			(type default)
-		)
-	)
-	(bus
-		(pts
 			(xy 209.55 132.08) (xy 213.36 132.08)
 		)
@@
 	(wire
 		(pts
+			(xy 257.81 97.79) (xy 257.81 99.06)
+		)
+		(stroke
+			(width 0)
+			(type default)
+		)
+	)
+	(wire
+		(pts
 			(xy 138.43 73.66) (xy 113.03 73.66)
 		)
@@
 	(wire
 		(pts
-			(xy 213.36 97.79) (xy 246.38 97.79)
+			(xy 213.36 95.25) (xy 246.38 95.25)
 		)
 		(stroke
@@
 	(wire
 		(pts
-			(xy 256.54 95.25) (xy 290.83 95.25)
+			(xy 256.54 92.71) (xy 290.83 92.71)
 		)
 		(stroke
@@
 	(wire
 		(pts
-			(xy 246.38 52.07) (xy 243.84 52.07)
+			(xy 101.6 187.96) (xy 102.87 187.96)
 		)
 		(stroke
@@
 	(bus
 		(pts
-			(xy 292.1 93.98) (xy 292.1 96.52)
+			(xy 292.1 88.9) (xy 292.1 93.98)
 		)
 		(stroke
@@
 		)
 	)
-	(wire
-		(pts
-			(xy 243.84 92.71) (xy 246.38 92.71)
-		)
-		(stroke
-			(width 0)
-			(type default)
-		)
-	)
 	(bus
 		(pts
@@
 		)
 	)
+	(wire
+		(pts
+			(xy 257.81 97.79) (xy 256.54 97.79)
+		)
+		(stroke
+			(width 0)
+			(type default)
+		)
+	)
 	(bus
 		(pts
@@
 	(wire
 		(pts
+			(xy 245.11 97.79) (xy 245.11 99.06)
+		)
+		(stroke
+			(width 0)
+			(type default)
+		)
+	)
+	(wire
+		(pts
 			(xy 77.47 43.18) (xy 102.87 43.18)
 		)
@@
 	(wire
 		(pts
-			(xy 102.87 198.12) (xy 100.33 198.12)
+			(xy 246.38 52.07) (xy 243.84 52.07)
 		)
 		(stroke
@@
 	(wire
 		(pts
-			(xy 100.33 193.04) (xy 102.87 193.04)
+			(xy 100.33 195.58) (xy 102.87 195.58)
 		)
 		(stroke
@@
 	(wire
 		(pts
-			(xy 259.08 92.71) (xy 256.54 92.71)
-		)
-		(stroke
-			(width 0)
-			(type default)
-		)
-	)
-	(wire
-		(pts
 			(xy 138.43 88.9) (xy 113.03 88.9)
 		)
@@
 	(wire
 		(pts
-			(xy 213.36 95.25) (xy 246.38 95.25)
+			(xy 213.36 92.71) (xy 246.38 92.71)
 		)
 		(stroke
@@
 	)
 	(label "DC_SCM_ESPI.IO3"
-		(at 267.97 95.25 0)
+		(at 267.97 92.71 0)
 		(effects
 			(font
@@
 	)
 	(label "DC_SCM_ESPI.IO0"
-		(at 236.22 97.79 180)
+		(at 236.22 95.25 180)
 		(effects
 			(font
@@
 	)
 	(label "DC_SCM_ESPI.~{RESET}"
-		(at 236.22 95.25 180)
+		(at 236.22 92.71 180)
 		(effects
 			(font
@@
 	)
 	(label "DC_SCM_ESPI.~{ALERT0}"
-		(at 267.97 97.79 0)
+		(at 267.97 95.25 0)
 		(effects
 			(font
@@
 	(hierarchical_label "DC_SCM_STBY_RDY"
 		(shape output)
-		(at 100.33 193.04 180)
+		(at 100.33 195.58 180)
 		(effects
 			(font
@@
 	(hierarchical_label "DC_SCM_12V_AUX"
 		(shape input)
-		(at 100.33 187.96 180)
+		(at 100.33 193.04 180)
 		(effects
 			(font
@@
 	(hierarchical_label "~{DC_SCM_STBY_RST}"
 		(shape input)
-		(at 100.33 195.58 180)
+		(at 100.33 198.12 180)
 		(effects
 			(font
@@
 	(hierarchical_label "~{DC_SCM_SPI_SCMCNTRL_IRQ0}"
 		(shape output)
-		(at 100.33 198.12 180)
+		(at 243.84 52.07 180)
 		(effects
 			(font
@@
 	(symbol
 		(lib_id "antmicropower:GND")
-		(at 243.84 92.71 270)
+		(at 245.11 99.06 0)
 		(unit 1)
 		(body_style 1)
@@
 		(dnp no)
 		(property "Reference" "#PWR023"
-			(at 241.3 101.6 0)
+			(at 254 101.6 0)
 			(hide yes)
 			(show_name no)
@@
 		)
 		(property "Value" "GND"
-			(at 241.046 92.71 90)
+			(at 245.11 101.854 0)
 			(show_name no)
 			(do_not_autoplace no)
@@
 					(thickness 0.15)
 				)
-				(justify right)
+				(justify top)
 			)
 		)
 		(property "Footprint" ""
-			(at 236.22 101.6 0)
+			(at 254 106.68 0)
 			(hide yes)
 			(show_name no)
@@
 		)
 		(property "Datasheet" ""
-			(at 231.14 101.6 0)
+			(at 254 111.76 0)
 			(hide yes)
 			(show_name no)
@@
 		)
 		(property "Description" ""
-			(at 228.6 101.6 0)
+			(at 254 114.3 0)
 			(hide yes)
 			(show_name no)
@@
 		)
 		(property "Author" "Antmicro"
-			(at 236.22 101.6 0)
+			(at 254 106.68 0)
 			(hide yes)
 			(show_name no)
@@
 		)
 		(property "License" "Apache-2.0"
-			(at 233.68 101.6 0)
+			(at 254 109.22 0)
 			(hide yes)
 			(show_name no)
@@
 	(symbol
 		(lib_id "antmicropower:GND")
-		(at 259.08 92.71 90)
+		(at 257.81 99.06 0)
 		(unit 1)
 		(body_style 1)
@@
 		(dnp no)
 		(property "Reference" "#PWR026"
-			(at 261.62 83.82 0)
+			(at 266.7 101.6 0)
 			(hide yes)
 			(show_name no)
@@
 		)
 		(property "Value" "GND"
-			(at 261.874 92.71 90)
+			(at 257.81 101.854 0)
 			(show_name no)
 			(do_not_autoplace no)
@@
 					(thickness 0.15)
 				)
-				(justify right)
+				(justify top)
 			)
 		)
 		(property "Footprint" ""
-			(at 266.7 83.82 0)
+			(at 266.7 106.68 0)
 			(hide yes)
 			(show_name no)
@@
 		)
 		(property "Datasheet" ""
-			(at 271.78 83.82 0)
+			(at 266.7 111.76 0)
 			(hide yes)
 			(show_name no)
@@
 		)
 		(property "Description" ""
-			(at 274.32 83.82 0)
+			(at 266.7 114.3 0)
 			(hide yes)
 			(show_name no)
@@
 		)
 		(property "Author" "Antmicro"
-			(at 266.7 83.82 0)
+			(at 266.7 106.68 0)
 			(hide yes)
 			(show_name no)
@@
 		)
 		(property "License" "Apache-2.0"
-			(at 269.24 83.82 0)
+			(at 266.7 109.22 0)
 			(hide yes)
 			(show_name no)
@@
 	(symbol
 		(lib_id "antmicropower:GND")
-		(at 243.84 52.07 270)
+		(at 101.6 187.96 270)
 		(unit 1)
 		(body_style 1)
@@
 		(dnp no)
 		(property "Reference" "#PWR022"
-			(at 241.3 60.96 0)
+			(at 99.06 196.85 0)
 			(hide yes)
 			(show_name no)
@@
 		)
 		(property "Value" "GND"
-			(at 241.046 52.07 90)
+			(at 98.806 187.96 90)
 			(show_name no)
 			(do_not_autoplace no)
@@
 		)
 		(property "Footprint" ""
-			(at 236.22 60.96 0)
+			(at 93.98 196.85 0)
 			(hide yes)
 			(show_name no)
@@
 		)
 		(property "Datasheet" ""
-			(at 231.14 60.96 0)
+			(at 88.9 196.85 0)
 			(hide yes)
 			(show_name no)
@@
 		)
 		(property "Description" ""
-			(at 228.6 60.96 0)
+			(at 86.36 196.85 0)
 			(hide yes)
 			(show_name no)
@@
 		)
 		(property "Author" "Antmicro"
-			(at 236.22 60.96 0)
+			(at 93.98 196.85 0)
 			(hide yes)
 			(show_name no)
@@
 		)
 		(property "License" "Apache-2.0"
-			(at 233.68 60.96 0)
+			(at 91.44 196.85 0)
 			(hide yes)
 			(show_name no)
