File: pcie_to_usb.kicad_sch (KiCad schematic)
At the start: 72 parts, among them J18 Molex_PicoBlade_1x4_0533980471, J19 Molex_PicoBlade_1x4_0533980471, J8 Tag-Connect_TC2050-IDC-NL_2x5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, U2 UPD720202K8-711-BAA-A, U5 W25Q80DV_USON, Y1 Resonator_24MHz_ECX-1247

Commit message: [#100720] Fix USB controller flash connection
Parts:
- R160: now fitted; now in the parts list
Connections:
- net SPI_DI: now also R156.2, R160.1, U5.5 (SI/IO0); no longer R157.2, R165.1, U5.2 (SO/IO1)
- net SPI_DO: now also R157.2, R165.1, U5.2 (SO/IO1); no longer R156.2, R160.1, U5.5 (SI/IO0)
- net USB_FLASH_SPI.DI: now also R156.1; no longer R157.1
- net USB_FLASH_SPI.DO: now also R157.1; no longer R156.1
Changed lines of the file:
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@@
 	)
 	(label "USB_FLASH_SPI.DO"
-		(at 90.17 240.03 180)
+		(at 90.17 242.57 180)
 		(effects
 			(font
@@
 	)
 	(label "USB_FLASH_SPI.DI"
-		(at 90.17 242.57 180)
+		(at 90.17 240.03 180)
 		(effects
 			(font
@@
 	)
 	(label "SPI_DI"
-		(at 146.05 242.57 180)
+		(at 146.05 240.03 180)
 		(effects
 			(font
@@
 	)
 	(label "SPI_DO"
-		(at 146.05 240.03 180)
+		(at 146.05 242.57 180)
 		(effects
 			(font
@@
 		(body_style 1)
 		(exclude_from_sim no)
-		(in_bom no)
+		(in_bom yes)
 		(on_board yes)
 		(in_pos_files yes)
-		(dnp yes)
+		(dnp no)
 		(property "Reference" "R160"
 			(at 106.68 229.87 90)

Commit message: [#100720] Add 0R to USB controller PCIe RX. Swap RX/TX
Parts:
- added R198, R199: R_0R_0402, antmicro-footprints:R_0402_1005Metric, symbol antmicroResistors0402:R_0R_0402
Connections:
- net DC-SCM_PCIE_LOCAL_USB.RX0+: now also C37.1; no longer U2.7 (PERXP)
- net DC-SCM_PCIE_LOCAL_USB.RX0-: now also C38.1; no longer U2.8 (PERXN)
- net DC-SCM_PCIE_LOCAL_USB.TX0+: now also R198.1; no longer C37.1
- net DC-SCM_PCIE_LOCAL_USB.TX0-: now also R199.1; no longer C38.1
- new net PERX+: R198.2, U2.7 (PERXP)
- new net PERX-: R199.2, U2.8 (PERXN)
