File: pcie_to_usb.kicad_sch (KiCad schematic)
At the start: 74 parts, among them J18 Molex_PicoBlade_1x4_0533980471, J19 Molex_PicoBlade_1x4_0533980471, J8 Tag-Connect_TC2050-IDC-NL_2x5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, U2 UPD720202K8-711-BAA-A, U5 W25Q80DV_USON, Y1 Resonator_24MHz_ECX-1247

Commit message: [#100720] Apply post review changes
Parts:
- removed R198, R199: R_0R_0402, antmicro-footprints:R_0402_1005Metric, symbol antmicroResistors0402:R_0R_0402
- added R132, R133, R141, R142, R143, R144: R_0R_0402, antmicro-footprints:R_0402_1005Metric, symbol antmicroResistors0402:R_0R_0402
Connections:
- net DC-SCM_PCIE_LOCAL_USB.RX0+: now also R132.2; no longer C37.1
- net DC-SCM_PCIE_LOCAL_USB.RX0-: now also R133.2; no longer C38.1
- net DC-SCM_PCIE_LOCAL_USB.TX0+: now also R141.2
- net DC-SCM_PCIE_LOCAL_USB.TX0-: now also R142.2
- net PERX+: now also R141.1
- net PERX-: now also R142.1
- net PETX+: now also C37.1, R132.1; no longer C37.2, U2.4 (PETXP)
- net PETX-: now also C38.1, R133.1; no longer C38.2, U2.5 (PETXN)
- net DC-SCM_CLK_100M_USB.CLK+ renamed PECLK+
- net PECLK+: now also R143.1
- net DC-SCM_CLK_100M_USB.CLK- renamed PECLK-
- net PECLK-: now also R144.1
- new net C_PETX+: C37.2, U2.4 (PETXP)
- new net C_PETX-: C38.2, U2.5 (PETXN)
- new net DC-SCM_CLK_100M_1.CLK+: R143.2
- new net DC-SCM_CLK_100M_1.CLK-: R144.2
