File: gold-fingers-connector.kicad_sch (KiCad schematic)
At the start: 128 parts, among them J1 Socket_DC-SCM-2.1_2x84_Rev-1-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

Commit message: [#100720] Apply post review changes
Parts:
- added R129, R130, R134, R138: R_0R_0402, antmicro-footprints:R_0402_1005Metric, symbol antmicroResistors0402:R_0R_0402
- R102, R103: now not fitted; now left out of the parts list
Connections:
- net DC_SCM_I2C_I3C16.SCL: now also R72.2; no longer R71.2
- net DC_SCM_I2C_I3C16.SDA: now also R71.2; no longer R72.2
- net PCIE_LOCAL_USB_RX0-: now reaches J1.A65 (PCIE_HPMROOT_SCM_HPM_5_DN)
- net PCIE_LOCAL_USB_RX0-: now also R138.1
- net PCIE_LOCAL_USB_RX0+: now reaches J1.A66 (PCIE_HPMROOT_SCM_HPM_5_DP)
- net PCIE_LOCAL_USB_RX0+: now also R134.1
- net PCIE_LOCAL_USB_TX0-: now reaches J1.B65 (PCIE_HPMROOT_HPM_SCM_5_DN)
- net PCIE_LOCAL_USB_TX0-: now also R130.1
- net PCIE_LOCAL_USB_TX0+: now reaches J1.B66 (PCIE_HPMROOT_HPM_SCM_5_DP)
- net PCIE_LOCAL_USB_TX0+: now also R129.1
- new net DC-SCM_PCIE_LOCAL_USB.RX0+: R134.2
- new net DC-SCM_PCIE_LOCAL_USB.RX0-: R138.2
- new net DC-SCM_PCIE_LOCAL_USB.TX0+: R129.2
- new net DC-SCM_PCIE_LOCAL_USB.TX0-: R130.2
- no-connect marks 4 -> 0
